File: hardware/proto1/ost-pid-proto1.kicad_sch (KiCad schematic)
At the start: 0 parts

Commit message: feat: add esp32s3 datasheet
Parts:
- added U1: ~, esp32-s3-tempel-lib:esp32-s3-tempel, symbol esp32-s3-tempel-lib:esp-32-s3-tempel
Changed lines of the file:
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@@
 	(generator_version "9.0")
 	(paper "A4")
+	(symbol
+		(lib_id "esp32-s3-tempel-lib:esp-32-s3-tempel")
+		(at 52.07 60.96 0)
+		(unit 1)
+		(exclude_from_sim no)
+		(in_bom yes)
+		(on_board yes)
+		(dnp no)
+		(fields_autoplaced yes)
+		(property "Reference" "U1"
+			(at 71.9933 44.45 0)
+			(effects
+				(font
+					(size 1.27 1.27)
+				)
+				(justify left)
+			)
+		)
+		(property "Value" "~"
+			(at 71.9933 46.99 0)
+			(effects
+				(font
+					(size 1.27 1.27)
+				)
+				(justify left)
+			)
+		)
+		(property "Footprint" "esp32-s3-tempel-lib:esp32-s3-tempel"
+			(at 52.07 60.96 0)
+			(effects
+				(font
+					(size 1.27 1.27)
+				)
+				(hide yes)
+			)
+		)
+		(property "Datasheet" ""
+			(at 52.07 60.96 0)
+			(effects
+				(font
+					(size 1.27 1.27)
+				)
+				(hide yes)
+			)
+		)
+		(property "Description" ""
+			(at 52.07 60.96 0)
+			(effects
+				(font
+					(size 1.27 1.27)
+				)
+				(hide yes)
+			)
+		)
+		(pin "16"
+		)
+		(pin "8"
+		)
+		(pin "27"
+		)
+		(pin "28"
+		)
+		(pin "22"
+		)
+		(pin "36"
+		)
+		(pin "25"
+		)
+		(pin "23"
+		)
+		(pin "30"
+		)
+		(pin "17"
+		)
+		(pin "12"
+		)
+		(pin "34"
+		)
+		(pin "1"
+		)
+		(pin "6"
+		)
+		(pin "24"
+		)
+		(pin "15"
+		)
+		(pin "2"
+		)
+		(pin "5"
+		)
+		(pin "4"
+		)
+		(pin "3"
+		)
+		(pin "31"
+		)
+		(pin "32"
+		)
+		(pin "19"
+		)
+		(pin "20"
+		)
+		(pin "21"
+		)
+		(pin "14"
+		)
+		(pin "29"
+		)
+		(pin "10"
+		)
+		(pin "35"
+		)
+		(pin "18"
+		)
+		(pin "33"
+		)
+		(pin "7"
+		)
+		(pin "9"
+		)
+		(pin "11"
+		)
+		(pin "26"
+		)
+		(pin "13"
+		)
+		(instances
+			(project ""
+				(path "/57ce6609-8746-4a6a-9ec1-053cec10b5d7"
+					(reference "U1")
+					(unit 1)
+				)
+			)
+		)
+	)
 	(sheet_instances
 		(path "/"
